File: library/SubcircuitLibrary/74HC157/74HC157.sch (KiCad schematic (older format))
At the start: 30 parts, among them U1 PORT, U10 d_and, U11 d_and, U12 d_and, U13 d_nor, U14 d_nor, U15 d_nor, U16 d_nor, U17 d_inverter, U18 d_inverter, U19 d_inverter, U2 d_inverter, U20 d_inverter, U3 d_and, U3 d_nor, U4 d_and, U4 d_nor, U5 d_and, U6 d_and, U7 d_and, U8 d_and, U9 d_and, X1 mux, X2 mux, X3 mux, X4 mux

Commit message: install script bypass 25.04 OS version check
Parts:
- removed U1: PORT, symbol PORT
- removed U10, U11, U12, U5, U6, U7, U8, U9: d_and, symbol d_and
- removed U13, U14, U15, U16, U3, U4: d_nor, symbol d_nor
- removed U17, U18, U19, U2, U20: d_inverter, symbol d_inverter
Connections:
- wire segments 70 -> 20
